File: hardware/LIONv3/LIONv3.kicad_pcb (KiCad board)
At the start: 4 copper layers, 50.1 x 85.2 mm, 89 parts, among them SW1 RESET, SW2 BOOT, U1 HC-1_25-2PWT, U10 E80-900M2213S, U11 W25Q16JVSSIQTR, U12 XL-1608UBC-04, U13 XL-1608UGC-04, U14 TPS259474ARPWR, U15 TLV76733DRVR, U16 XL-1608SURC-06, U17 INA226AIDGSR, U18 HC-1_25-2PWT, U19 HC-1_25-2PWT, U2 HC-1_25-2PWT, U20 HC-1_25-2PWT, U21 TCAN3414DR, U3 ESP32-C6-MINI-1-N4, U5 HC-1_25-2PWT, U6 TMP112AIDRLR, U7 USBLC6-2SC6, U8 TYPE-C_16PIN_2MD(073), U9 INA226AIDGSR

Commit message: refactor(hardware): improve schematic
Parts:
- moved U20 0.75 mm to (364.8, 85.1)
Routing:
- net GND: track 13.7 -> 13.3 mm, vias 383 -> 386
Other:
- board text added: "CAN"

Commit message: feat(hardware): adapt PCB layout to Mini version
Parts:
- removed the G*** at (341.0, 120.2)
Routing:
- net GND: vias 386 -> 391
Other:
- board size 50.1 x 85.2 mm -> 50.1 x 40.1 mm

Commit message: feat(hardware): improve silkscreen positioning
Parts:
- removed U1, U18, U19, U2, U20, U5: HC-1_25-2PWT, LIONv3-Footprints:CONN-SMD_2P-P1.25-HC-1.25-2PWT
- removed U12: XL-1608UBC-04, LIONv3-Footprints:LED0603-RD_BLUE
- removed U13: XL-1608UGC-04, LIONv3-Footprints:LED0603-RD_GREEN
- removed U16: XL-1608SURC-06, LIONv3-Footprints:LED0603-RD_RED
- added D5: PMEG2010ER, Diode_SMD:Nexperia_CFP3_SOD-123W, F.Cu at (8.87, 1.12)
- added D7: LED, LED_SMD:LED_0603_1608Metric, F.Cu at (332.9, 90.6)
- added D8: LED, LED_SMD:LED_0603_1608Metric, F.Cu at (332.9, 87.8)
- added D9: LED, LED_SMD:LED_0603_1608Metric, F.Cu at (332.9, 93.4)
- added FB2: BLM21PG221SN1D, Inductor_SMD:L_0805_2012Metric, F.Cu at (8.32, 4.12)
- added H1: MountingHole_Pad, MountingHole:MountingHole_2.5mm, F.Cu at (2.77, 2.77)
- added H2: MountingHole_Pad, MountingHole:MountingHole_2.5mm, F.Cu at (2.77, 9.32)
- added H3: MountingHole_Pad, MountingHole:MountingHole_2.5mm, F.Cu at (2.77, 15.9)
- added J1: 532610271, LIONv3-Footprints:CONN-SMD_532610271, B.Cu at (322.3, 76.6)
- added J2: 532610271, LIONv3-Footprints:CONN-SMD_532610271, B.Cu at (364.8, 89.1)
- added J3: 532610271, LIONv3-Footprints:CONN-SMD_532610271, B.Cu at (364.8, 70.0)
- added J4: 532610271, LIONv3-Footprints:CONN-SMD_532610271, B.Cu at (322.3, 67.7)
- added J5: 532610271, LIONv3-Footprints:CONN-SMD_532610271, B.Cu at (364.8, 79.8)
- added TP1: TestPoint_Square, TestPoint:TestPoint_Pad_D1.5mm, F.Cu at (253.7, 81.7)
- added TP10: TestPoint_Square, TestPoint:TestPoint_Pad_D1.5mm, F.Cu at (267.9, 62.0)
- added TP11: TestPoint_Square, TestPoint:TestPoint_Pad_D1.5mm, F.Cu at (267.9, 65.6)
- added TP12: TestPoint_Square, TestPoint:TestPoint_Pad_D1.5mm, F.Cu at (267.9, 69.1)
- added TP2: TestPoint_Square, TestPoint:TestPoint_Pad_D1.5mm, F.Cu at (253.7, 85.2)
- added TP3: TestPoint_Square, TestPoint:TestPoint_Pad_D1.5mm, F.Cu at (253.7, 88.8)
- added TP4: TestPoint_Square, TestPoint:TestPoint_Pad_D1.5mm, F.Cu at (253.7, 92.3)
- added TP5: TestPoint_Square, TestPoint:TestPoint_Pad_D1.5mm, F.Cu at (257.3, 81.7)
- added TP6: TestPoint_Square, TestPoint:TestPoint_Pad_D1.5mm, F.Cu at (257.3, 85.2)
- added TP7: TestPoint_Square, TestPoint:TestPoint_Pad_D1.5mm, F.Cu at (257.3, 88.8)
- added TP8: TestPoint_Square, TestPoint:TestPoint_Pad_D1.5mm, F.Cu at (267.9, 74.7)
- added TP9: TestPoint_Square, TestPoint:TestPoint_Pad_D1.5mm, F.Cu at (267.9, 78.2)
- moved G*** 27.0 mm to (361.1, 62.9)
- moved R28 16.7 mm to (377.9, 63.8)
- moved D6 16.7 mm to (376.8, 66.5)
- moved R29 16.7 mm to (375.7, 63.8)
- moved D5 1.75 mm to (329.8, 79.5)
- moved FB2 1.75 mm to (327.6, 77.6)
Routing:
- net /CAN_P: track 11.9 -> 0.00 mm
- net /CAN_N: track 11.3 -> 0.00 mm
- net /TMP_ALERT: track 34.7 -> 27.4 mm
- net /CAN_STB: track 33.1 -> 27.7 mm
- net /CAN_RX: track 27.7 -> 26.3 mm
- net /CAN_TX: track 20.5 -> 19.4 mm
- net GND: vias 391 -> 386
Other:
- board text added: "+"
- board text added: "+3V"
- board text added: "-"
- board text added: "C"
- board text added: "D"
- board text added: "H"
- board text added: "L"
- board text removed: "+3.3V"
- board text removed: "GND"
