File: hardware/LIONv3/LIONv3.kicad_pcb (KiCad board)
At the start: 4 copper layers, 50.1 x 40.1 mm, 104 parts, among them J1 532610271, J2 532610271, J3 532610271, J4 532610271, J5 532610271, SW1 RESET, SW2 BOOT, U10 E80-900M2213S, U11 W25Q16JVSSIQTR, U14 TPS259474ARPWR, U15 TLV76733DRVR, U17 INA226AIDGSR, U21 TCAN3414DR, U3 ESP32-C6-MINI-1-N4, U6 TMP112AIDRLR, U7 USBLC6-2SC6, U8 TYPE-C_16PIN_2MD(073), U9 INA226AIDGSR

Commit message: feat(hardware): finish LIONv3-Mini routing
Parts:
- removed the D5 at (8.87, 1.12)
- removed the FB2 at (8.32, 4.12)
- removed the H1 at (2.77, 2.77)
- removed the H2 at (2.77, 9.32)
- removed the H3 at (2.77, 15.9)
- removed TP1, TP10, TP11, TP12, TP2, TP3, TP4, TP5, TP6, TP7, TP8, TP9: TestPoint_Square, TestPoint:TestPoint_Pad_D1.5mm
- added G***: LOGO, LOGO, B.Cu at (343.4, 77.7)
- moved D6 19.7 mm to (357.4, 70.0), turned to 180 degrees
- moved R28 19.4 mm to (360.0, 71.1), turned to -90 degrees
- moved R29 16.4 mm to (360.0, 68.9), turned to -90 degrees
- moved J2 9.57 mm to (364.8, 79.5)
- moved J5 9.27 mm to (364.8, 89.1)
- moved U21 3.00 mm to (351.4, 70.0)
- moved C20 2.85 mm to (345.7, 70.0)
- moved C21 2.85 mm to (347.3, 70.0)
- moved R15 1.58 mm to (346.4, 67.4)
- moved D5 0.83 mm to (329.7, 80.3)
- moved FB2 0.20 mm to (327.4, 77.6)
Connections:
- J5 pad 1: /I2C_SCL -> /I2C_SDA
- J5 pad 2: /I2C_SDA -> /I2C_SCL
Routing:
- net /CAN_P: track 0.00 -> 10.0 mm
- net /CAN_N: track 0.00 -> 9.99 mm
- net Net-(JP1-A): track 2.29 -> 10.8 mm
- net /TMP_ALERT: track 27.4 -> 34.7 mm
- net Net-(JP1-B): track 2.30 -> 6.85 mm
- net /CAN_STB: track 27.7 -> 30.6 mm
- net /I2C_SCL: track 63.3 -> 65.5 mm
- net Net-(U11-IO3): track 0.00 -> 1.63 mm
- net /CAN_TX: track 19.4 -> 18.0 mm
- net +3.3V: track 21.0 -> 19.7 mm, vias 32 -> 27
- net /SPI_SCK: track 28.7 -> 29.8 mm
- net GND: track 13.3 -> 12.2 mm, vias 386 -> 379
- net /SPI_PICO: track 29.3 -> 30.3 mm
- net /I2C_SDA: track 66.0 -> 66.9 mm
Other:
- board text added: "LionV3-Mini"
- board text added: "v1•343200bf"
- board text removed: "v1•e8e3db53"

Commit message: feat(hardware): finish LIONv3-Mini rev1.0
Parts:
- J1, J2, J3, J4, J5: footprint LIONv3-Footprints:CONN-SMD_532610271 -> LIONv3-Footprints:Molex_PicoBlade_53261-0271_1x02-1MP_P1.25mm_Horizontal
- SW1: value RESET -> ~
- SW2: value BOOT -> ~
- moved J1 203.1 mm to (120.7, 101.2), turned to 90 degrees
- moved J4 203.0 mm to (120.7, 91.6), turned to 90 degrees
- moved FB2 202.0 mm to (126.8, 102.0)
- moved G*** 202.0 mm to (142.9, 101.7)
- moved C17 202.0 mm to (143.1, 115.7)
- moved C22 202.0 mm to (159.0, 84.3)
- moved C3 202.0 mm to (121.5, 98.9)
- moved C4 202.0 mm to (163.5, 97.5)
- moved C8 202.0 mm to (161.1, 117.9)
- moved D3 202.0 mm to (130.5, 110.8)
- moved H3 202.0 mm to (120.7, 118.8)
- moved R1 202.0 mm to (121.3, 93.1)
- moved R10 202.0 mm to (123.0, 112.9)
- moved R12 202.0 mm to (156.0, 110.2)
- moved R13 202.0 mm to (145.5, 98.6)
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Connections:
- U10 pad 15: /RF/ANT_915 -> unconnected-(U10-ANT_915-Pad15)
Routing:
- net /I2C_SDA: track 66.9 -> 65.4 mm
- net +3.3V: track 19.7 -> 18.6 mm
- net /CAN_RX: track 26.3 -> 27.2 mm
- net Net-(JP1-A): track 10.8 -> 10.1 mm
- net Net-(U11-IO3): track 1.63 -> 0.93 mm
- net GND: vias 379 -> 380
Other:
- board size 50.1 x 40.1 mm -> 50.2 x 40.2 mm
