File: hardware/LIONv3/CANbus.kicad_sch (KiCad schematic)
At the start: 8 parts, among them U21 TCAN3414DR

Commit message: refactor(hardware): improve schematic
Parts:
- R28, R29: LCSC (none) -> C227152
Changed lines of the file:
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@@
+			)
+		)
+		(property "LCSC" "C227152"
+			(at 139.7 31.75 90)
+			(hide yes)
+			(show_name no)
+			(do_not_autoplace no)
+			(effects
+				(font
+					(size 1.27 1.27)
+				)
 			)
 		)
@@
 			(hide yes)
 			(show_name no)
+			(do_not_autoplace no)
+			(effects
+				(font
+					(size 1.27 1.27)
+				)
+			)
+		)
+		(property "LCSC" "C227152"
+			(at 163.83 31.75 90)
+			(hide yes)
+			(show_name no)
