File: hardware/LIONv3/POWER.kicad_sch (KiCad schematic)
At the start: 31 parts, among them U13 XL-1608UGC-04, U14 TPS259474ARPWR, U15 TLV76733DRVR, U16 XL-1608SURC-06, U17 INA226AIDGSR, U18 HC-1_25-2PWT, U19 HC-1_25-2PWT, U20 HC-1_25-2PWT

Commit message: refactor(hardware): improve schematic
Other:
- moved on the sheet: D5, FB2, U18, U19, U20

Commit message: feat(hardware): improve silkscreen positioning
Parts:
- removed D5: PMEG2010ER, Diode_SMD:Nexperia_CFP3_SOD-123W, symbol Diode:PMEG2010ER
- removed FB2: BLM21PG221SN1D, Inductor_SMD:L_0805_2012Metric, symbol Device:FerriteBead_Small
- removed U13: XL-1608UGC-04, LIONv3-Footprints:LED0603-RD_GREEN, symbol LIONv3-Symbols:XL-1608UGC-04
- removed U16: XL-1608SURC-06, LIONv3-Footprints:LED0603-RD_RED, symbol LIONv3-Symbols:XL-1608SURC-06
- removed U18, U19, U20: HC-1_25-2PWT, LIONv3-Footprints:CONN-SMD_2P-P1.25-HC-1.25-2PWT, symbol LIONv3-Symbols:HC-1_25-2PWT
- added D7, D8: LED, LED_SMD:LED_0603_1608Metric, symbol Device:LED
Connections:
- net GND: now also D8.1 (K)
- net LED_FAULT: now also D7.1 (K)
- net at R20.1: now also D8.2 (A)
- net at R24.1: now also D7.2 (A)

Commit message: feat(hardware): finish LIONv3-Mini rev1.0
Parts:
- removed TP10, TP11, TP12: TestPoint_Square, TestPoint:TestPoint_Pad_D1.5mm, symbol Connector:TestPoint_Square
Other:
- note removed: "LATCH CONNECTORS (NO reverse-polarity) mates in one orientation only"
