File: hardware/LIONv3/RF.kicad_sch (KiCad schematic)
At the start: 19 parts, among them U10 E80-900M2213S, U11 W25Q16JVSSIQTR, U12 XL-1608UBC-04, U9 INA226AIDGSR

Commit message: feat(hardware): improve silkscreen positioning
Parts:
- removed U12: XL-1608UBC-04, LIONv3-Footprints:LED0603-RD_BLUE, symbol LIONv3-Symbols:XL-1608UBC-04
- added D9: LED, LED_SMD:LED_0603_1608Metric, symbol Device:LED
Connections:
- net GND: now also D9.1 (K)
- net at R17.1: now also D9.2 (A)
Changed lines of the file:
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@@
 	(wire
 		(pts
-			(xy 62.23 92.71) (xy 71.12 92.71)
+			(xy 62.23 92.71) (xy 73.66 92.71)
 		)
 		(stroke
@@
 	)
 	(symbol
-		(lib_name "XL-1608UBC-04_1")
-		(lib_id "LIONv3-Symbols:XL-1608UBC-04")
-		(at 76.2 92.71 0)
+		(lib_id "Device:LED")
+		(at 77.47 92.71 0)
 		(unit 1)
 		(body_style 1)
@@
 		(dnp no)
 		(fields_autoplaced yes)
-		(property "Reference" "U12"
-			(at 75.438 83.82 0)
+		(property "Reference" "D9"
+			(at 75.8825 86.36 0)
 			(show_name no)
 			(do_not_autoplace no)
@@
 			)
 		)
-		(property "Value" "XL-1608UBC-04"
-			(at 75.438 86.36 0)
+		(property "Value" "LED"
+			(at 75.8825 88.9 0)
 			(show_name no)
 			(do_not_autoplace no)
@@
 			)
 		)
-		(property "Footprint" "LIONv3-Footprints:LED0603-RD_BLUE"
-			(at 76.2 102.87 0)
+		(property "Footprint" "LED_SMD:LED_0603_1608Metric"
+			(at 77.47 92.71 0)
 			(hide yes)
 			(show_name no)
@@
 				(font
 					(size 1.27 1.27)
-					(italic yes)
 				)
 			)
 		)
 		(property "Datasheet" "file://${KIPRJMOD}/LIONv3-Datasheets/XL-1608UBC-04.pdf"
-			(at 73.914 92.583 0)
+			(at 77.47 92.71 0)
 			(hide yes)
 			(show_name no)
@@
 					(size 1.27 1.27)
 				)
-				(justify left)
 			)
 		)
-		(property "Description" ""
-			(at 76.2 92.71 0)
+		(property "Description" "Light emitting diode"
+			(at 77.47 92.71 0)
+			(hide yes)
+			(show_name no)
+			(do_not_autoplace no)
+			(effects
+				(font
+					(size 1.27 1.27)
+				)
+			)
+		)
+		(property "Sim.Pins" "1=K 2=A"
+			(at 77.47 92.71 0)
 			(hide yes)
 			(show_name no)
@@
 		)
 		(property "LCSC" "C965807"
-			(at 76.2 92.71 0)
+			(at 77.47 92.71 0)
 			(hide yes)
 			(show_name no)
@@
 			(project "LIONv3"
 				(path "/3cc9e06f-00d0-4bec-822f-2e156022ced4/d6030e6b-69d2-4923-80e2-2aab4b335fec"
-					(reference "U12")
+					(reference "D9")
 					(unit 1)
 				)

Commit message: feat(hardware): finish LIONv3-Mini rev1.0
Parts:
- removed AE1: Antenna, symbol Device:Antenna
- removed TP8, TP9: TestPoint_Square, TestPoint:TestPoint_Pad_D1.5mm, symbol Connector:TestPoint_Square
Connections:
- net ANT_915: no longer names the net of U10.15 (ANT_915)
- no-connect marks 4 -> 5
Other:
- moved on the sheet: D9, R17
